File: SteeringAngleModule.kicad_sch (KiCad schematic)
At the start: 6 parts, among them J1 Conn_01x03_Socket, J2 Conn_01x03_Socket, J3 Conn_01x04_Socket, U1 MCP3423

Commit message: update
Parts:
- removed JP1, JP2: SolderJumper_2_Open, TestPoint:TestPoint_2Pads_Pitch2.54mm_Drill0.8mm, symbol Jumper:SolderJumper_2_Open
- added C1: 0.1uF, symbol Device:C
- added C2: 10uF, symbol Device:C
- added D1: PowerLED, symbol Device:LED
- added JP1, JP2: SolderJumper_3_Open, symbol Jumper:SolderJumper_3_Open
- added R1: 330, symbol Device:R
- added R4, R5: 5k, symbol Device:R
- added R6, R8: 1k, symbol Device:R
- added R7, R9: 2k, symbol Device:R
Connections:
- net +3.3VADC: now also C1.1, C2.1, D1.2 (A), JP1.1 (A), JP2.1 (A), R4.1, R5.1
- net GNDA: now also C1.2, C2.2, JP1.3 (B), JP2.3 (B), R1.2, R7.2, R9.2; no longer U1.10 (A1), U1.9 (A0)
- net SCL: now also R4.2
- net SDA: now also R5.2
- removed net OUT+: J1.2 (Pin_2), J2.2 (Pin_2), U1.1 (CH1+), U1.4 (CH2+)
- new net: D1.1 (K), R1.1
- new net A0: JP2.2 (C), U1.9 (A0)
- new net A1: JP1.2 (C), U1.10 (A1)
- new net CH1+: R6.2, R7.1, U1.1 (CH1+)
- new net CH2+: R8.2, R9.1, U1.4 (CH2+)
- new net OUT+_ele: J1.2 (Pin_2), R8.1
- new net OUT+_ladder: J2.2 (Pin_2), R6.1
Other:
- note added: "A0,A1: Addr_Low (VSS<=v<=0.2Vdd) A0,A1: Addr_High (0.75Vdd<=v<=Vdd)"
- note added: "SCL および SDAのプルアップ抵抗値の標準レンジは、 標準モード (100 kHz) およびファースト モード (400 kHz)で5～10 kΩ、ハイスピード モード(3.4 MHz) で 1 kΩ 未満です。"
- note added: "↖電通大生ｗ"
- note added: "入力電圧レンジ, Vin:差動電圧, Vincom:コモンノード電圧 VIN = (CHn+) - (CHn-) VINCOM = ((CHn+) + (CHn-))/2 内部基準電圧Vref=2.048V"
- moved on the sheet: J1, J2, J3, U1

Commit message: update
Parts:
- added R2: 1k, Resistor_SMD:R_0603_1608Metric, symbol Device:R
- added R3: 2k, Resistor_SMD:R_0603_1608Metric, symbol Device:R
- C1: value 0.1uF -> 10uF
- C2: value 10uF -> 0.1uF
- D1: footprint (none) -> LED_SMD:LED_0603_1608Metric
- R1: value 330 -> 1k; footprint (none) -> Resistor_SMD:R_0603_1608Metric
- R4, R5: value 5k -> 5.1k; footprint (none) -> Resistor_SMD:R_0603_1608Metric
- R6, R7, R8: footprint (none) -> Resistor_SMD:R_0603_1608Metric
Connections:
- net +3.3VADC: now also R2.1; no longer J1.1 (Pin_1), J2.1 (Pin_1)
- net CH1+: now also J1.2 (Pin_2)
- net CH2+: now also J2.2 (Pin_2)
- net GNDA: now also R3.2
- net OUT+_ele: no longer J1.2 (Pin_2)
- net OUT+_ladder: no longer J2.2 (Pin_2)
- new net input_ele: J1.1 (Pin_1), J2.1 (Pin_1), R2.2, R3.1
Other:
- note removed: "↖電通大生ｗ"
- moved on the sheet: R4, R5

Commit message: update
Parts:
- removed R2, R6, R8: 1k, Resistor_SMD:R_0603_1608Metric, symbol Device:R
- removed R3, R7: 2k, Resistor_SMD:R_0603_1608Metric, symbol Device:R
- removed R9: 2k, symbol Device:R
- added C3, C4: 1u, symbol Device:C
- added U2: MCP1700T-1802E/TT, Package_TO_SOT_SMD:SOT-89-3, symbol Regulator_Linear:MCP1700x-180xxMB
- D1: value PowerLED -> indicator
- J1: value Conn_01x03_Socket -> Elevator
- J2: value Conn_01x03_Socket -> Ladder
Connections:
- net +3.3VADC: no longer C1.1, C2.1, D1.2 (A), J3.1 (Pin_1), R4.1, R5.1, U1.6 (Vdd)
- net GNDA: now also C3.2, C4.2, U2.1 (GND)
- net A0: no longer names the net of JP2.2 (C), U1.9 (A0)
- net A1: no longer names the net of JP1.2 (C), U1.10 (A1)
- net input_ele renamed +1V8
- net +1V8: now also C4.1, U2.3 (VO)
- new net +3.3V: C1.1, C2.1, C3.1, D1.2 (A), J3.1 (Pin_1), R4.1, R5.1, U1.6 (Vdd), U2.2 (VI)
Other:
- moved on the sheet: C1, C2, D1, J1, J2, J3, JP2, R1, R4, R5, U1
